Commit message: robot_arm added

File: my_robot_description/urdf/common_properties.xacro (robot description, xacro)
@@ -6,4 +6,10 @@
     <material name="grey">
         <color rgba="0.5 0.5 0.5 1" />
+    </material>
+    <material name="orange">
+        <color rgba="1.0 0.5 0.0 1" />
+    </material>
+    <material name="yellow">
+        <color rgba="1.0 1.0 0.0 1" />
     </material>
     <xacro:macro name="box_inertia" params="m l w h xyz rpy">

File: my_robot_description/urdf/mobile_base.xacro (robot description, xacro)
@@ -20,5 +20,5 @@
             <origin xyz="0 0 ${base_height / 2.0}" rpy="0 0 0" />
         </collision>
-        <xacro:box_inertia m="5.0" l="${base_length}" w="${base_width}" h="${base_height}"
+        <xacro:box_inertia m="5.0" w="${base_length}" h="${base_width}" l="${base_height}"
                            xyz="0 0 ${base_height / 2.0}" rpy="0 0 0" />
     </link>

File: my_robot_description/urdf/my_robot.urdf.xacro (robot description, xacro)
@@ -2,5 +2,11 @@
 <robot name="my_robot" xmlns:xacro="http://www.ros.org/wiki/xacro">
     <xacro:include filename="common_properties.xacro" />
+    <xacro:include filename="robot_arm.xacro" />
     <xacro:include filename="mobile_base.xacro" />
     <xacro:include filename="camera.xacro" />
+    <joint name="base_arm_joint" type="fixed">
+        <parent link="base_link" />
+        <child link="arm_base_link" />
+        <origin xyz="${base_length / 3.0} 0 ${base_height}" rpy="0 0 0" />
+    </joint>
 </robot>
